Commit message: Added the camera to the bot.

File: description/color.xacro (robot description, xacro)
@@ -13,3 +13,6 @@
         <color rgba="0 0 0 1"/>
     </material>
+    <material name="red">
+        <color rgba="1 0 0 1"/>
+    </material>
 </robot>

File: description/gazebo.xacro (robot description, xacro)
@@ -15,3 +15,21 @@
         <mu2 value="0.001"/>
     </gazebo>
+    <gazebo>
+        <plugin name = "diff_drive" filename="libgazebo_ros_diff_drive.so">
+            <!-- WHeel Information-->
+            <left_joint>left_wheel_joint</left_joint>
+            <right_joint>right_wheel_joint</right_joint>
+            <wheel_separation>0.35</wheel_separation>
+            <wheel_diameter>0.1</wheel_diameter>
+            <!-- limits-->
+            <max_wheel_torque>200</max_wheel_torque>
+            <max_wheel_acceleration>10</max_wheel_acceleration>
+            <!-- Output-->
+            <odometry_frame>odom</odometry_frame>
+            <robot_base_frame>base_link</robot_base_frame>
+            <publish_odom>true</publish_odom>
+            <publish_odom_tf>true</publish_odom_tf>
+            <publish_wheel_tf>true</publish_wheel_tf>
+        </plugin>
+    </gazebo>
 </robot>

File: description/robot.urdf.xacro (robot description, xacro)
@@ -3,3 +3,5 @@
    <xacro:include filename="robot_core.xacro" />
    <xacro:include filename="gazebo.xacro" />
+   <xacro:include filename="lidar.xacro"/>
+   <xacro:include filename="camera.xacro"/>
 </robot>
