Commit message: SLAM and NAV

File: description/lidar.xacro (robot description, xacro)
@@ -44,5 +44,5 @@
             <plugin name = "laser_controller" filename = "libgazebo_ros_ray_sensor.so">
                 <ros>
-                    <argument>-/output:=scan</argument>
+                    <argument>~/out:=scan</argument>
                 </ros>
                 <output_type>sensor_msgs/LaserScan</output_type>

File: description/robot.urdf.xacro (robot description, xacro)
@@ -8,5 +8,5 @@
    </xacro:if>
    <xacro:unless value="$(arg use_ros2_control)">
-      <xacro:include filename="gazebo_control.xacro" />
+      <xacro:include filename="gazebo.xacro" />
    </xacro:unless>
    <xacro:if value="$(arg use_camera)">

File: description/robot_core.xacro (robot description, xacro)
@@ -4,4 +4,11 @@
     <xacro:include filename="inertial_macros.xacro" />
     <link name="base_link">
+    </link>
+    <joint name="base_footprint_joint" type="fixed">
+        <parent link="base_link"/>
+        <child link="base_footprint"/>
+        <origin xyz="0 0 0" rpy="0 0 0"/>
+    </joint>
+    <link name = "base_footprint">
     </link>
     <!-- CHASSIS-->
